File: PCB/master_schematic.brd (EAGLE design)
At the start: 40 x 80 mm, 17 parts, among them IC1 7805T, J1 I2C_OUT_1, J2 I2C_OUT_2, Q1 2N7000KL/BS170KL, Q2 2N7000KL/BS170KL, X1 12V

Commit message: new versions of pcb
Parts:
- added C1, C2: 100nF, rcl:C025-030X050
- moved U$2 20.4 mm to (-2.54, 67.3)
- moved IC1 1.27 mm to (5.08, 8.89)
Connections:
- net +5V: now also C2.1
- net GND: now also C1.2, C2.2
- net N$4: now also C1.1
Routing:
- net GND: track 151.4 -> 171.8 mm
- net N$9: track 12.2 -> 32.6 mm
- net N$5: track 27.8 -> 47.1 mm
- net N$14: track 72.4 -> 53.5 mm
- net +5V: track 139.4 -> 150.0 mm
- net N$4: track 11.5 -> 16.5 mm
Other:
- board text added: "Split Flap Master v1.1"
