File: PCB/master_schematic.sch (EAGLE design)
At the start: 17 parts, among them IC1 7805T, J1 I2C_OUT_1, J2 I2C_OUT_2, Q1 2N7000KL/BS170KL, Q2 2N7000KL/BS170KL, X1 12V

Commit message: new versions of pcb
Parts:
- added C1, C2: 100nF, rcl:C-EU025-030X050
Connections:
- net +5V: now also C2.1
- net GND: now also C1.2, C2.2
- net N$4: now also C1.1
Changed lines of the file:
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@@
 <part name="R7" library="rcl" library_urn="urn:adsk.eagle:library:334" deviceset="R-EU_" device="0207/10" package3d_urn="urn:adsk.eagle:package:23491/1" value="4k7"/>
 <part name="R8" library="rcl" library_urn="urn:adsk.eagle:library:334" deviceset="R-EU_" device="0207/10" package3d_urn="urn:adsk.eagle:package:23491/1" value="4k7"/>
+<part name="C1" library="rcl" library_urn="urn:adsk.eagle:library:334" deviceset="C-EU" device="025-030X050" package3d_urn="urn:adsk.eagle:package:23631/1" value="100nF"/>
+<part name="C2" library="rcl" library_urn="urn:adsk.eagle:library:334" deviceset="C-EU" device="025-030X050" package3d_urn="urn:adsk.eagle:package:23631/1" value="100nF"/>
 </parts>
 <sheets>
@@
 <attribute name="VALUE" x="-51.562" y="153.67" size="1.778" layer="96" rot="R270"/>
 </instance>
+<instance part="C1" gate="G$1" x="-71.12" y="119.38" smashed="yes">
+<attribute name="NAME" x="-69.596" y="119.761" size="1.778" layer="95"/>
+<attribute name="VALUE" x="-69.596" y="114.681" size="1.778" layer="96"/>
+</instance>
+<instance part="C2" gate="G$1" x="12.7" y="167.64" smashed="yes">
+<attribute name="NAME" x="14.224" y="168.021" size="1.778" layer="95"/>
+<attribute name="VALUE" x="14.224" y="162.941" size="1.778" layer="96"/>
+</instance>
 </instances>
 <busses>
@@
 <wire x1="-78.74" y1="114.3" x2="-78.74" y2="109.22" width="0.1524" layer="91"/>
 <pinref part="IC1" gate="A1" pin="GND"/>
-<wire x1="-55.88" y1="114.3" x2="-78.74" y2="114.3" width="0.1524" layer="91"/>
+<wire x1="-55.88" y1="114.3" x2="-71.12" y2="114.3" width="0.1524" layer="91"/>
 <junction x="-78.74" y="114.3"/>
 <pinref part="U$1" gate="G$1" pin="GND"/>
+<wire x1="-71.12" y1="114.3" x2="-78.74" y2="114.3" width="0.1524" layer="91"/>
 <wire x1="-35.56" y1="127" x2="-38.1" y2="127" width="0.1524" layer="91"/>
 <wire x1="-38.1" y1="127" x2="-38.1" y2="114.3" width="0.1524" layer="91"/>
@@
 <wire x1="-55.88" y1="73.66" x2="-55.88" y2="86.36" width="0.1524" layer="91"/>
 <junction x="-55.88" y="86.36"/>
+<pinref part="C1" gate="G$1" pin="2"/>
+<junction x="-71.12" y="114.3"/>
 </segment>
 <segment>
@@
 <pinref part="U$3" gate="G$1" pin="GND"/>
 <pinref part="GND3" gate="1" pin="GND"/>
+<pinref part="C2" gate="G$1" pin="2"/>
+<wire x1="12.7" y1="162.56" x2="27.94" y2="162.56" width="0.1524" layer="91"/>
+<junction x="27.94" y="162.56"/>
 </segment>
 </net>
@@
 <wire x1="-76.2" y1="157.48" x2="-76.2" y2="121.92" width="0.1524" layer="91"/>
 <pinref part="IC1" gate="A1" pin="VI"/>
-<wire x1="-76.2" y1="121.92" x2="-66.04" y2="121.92" width="0.1524" layer="91"/>
+<wire x1="-76.2" y1="121.92" x2="-71.12" y2="121.92" width="0.1524" layer="91"/>
+<pinref part="C1" gate="G$1" pin="1"/>
+<wire x1="-71.12" y1="121.92" x2="-66.04" y2="121.92" width="0.1524" layer="91"/>
+<junction x="-71.12" y="121.92"/>
 </segment>
 </net>
@@
 <pinref part="P+2" gate="1" pin="+5V"/>
 <wire x1="12.7" y1="170.18" x2="12.7" y2="172.72" width="0.1524" layer="91"/>
-</segment>
-<segment>
+<pinref part="C2" gate="G$1" pin="1"/>
+<junction x="12.7" y="170.18"/>
+</segment>
+<segment>
