File: PCB/unit_schematic_1_1.brd (EAGLE design)
At the start: 43 x 80 mm, 8 parts, among them IC1 ULN2003AN, IC2 7805T, J1 HALL, J2 I2C_IN, J3 I2C_OUT, X1 28BYJ48, X2 12V

Commit message: new versions of pcb
Parts:
- removed J1: HALL, SparkFun-Connectors:JST-3-PTH
- added R1: 100K, rcl:0207/10
- added X3: Sensors, Rembrandt Electronics - JST XH Connectors v1-0:JST-XH-05-PACKAGE-ROUND-PAD
Connections:
- removed net N$10: IC2.3, J1.1, U$2.RAW
- new net +5V: IC2.3, R1.2, U$2.RAW, X3.1
- new net N$2: R1.1, U$2.A0, X3.5
- net GND: now also X3.2, X3.4; no longer J1.2
- net N$11: now also X3.3; no longer J1.3
Routing:
- net +5V: track 0.00 -> 64.4 mm
- net N$10: track 58.2 -> 0.00 mm
- net N$2: track 0.00 -> 34.8 mm
- net GND: track 114.1 -> 119.3 mm
- net N$11: track 16.9 -> 21.7 mm
Other:
- board text added: "Split Flap Unit v1.1"
